File: 05-Layout/nowae026/nowae026-0/nowae026.kicad_pcb (KiCad board)
At the start: 2 copper layers, 22.9 x 34.3 mm, 6 parts, among them J1 JUMPER-2, J2 JUMPER-2, P1 CONN, U1 BGM111A256V21

Commit message: WiP on PCB (nowae026)
Parts:
- added G***: LOGO, LOGO:LOGO_NOWAE_15MM_FSILK, F.Cu at (147.2, 83.5)
- added G***: LOGO, LOGO:LOGO_NOWAE_20MM_FSILK, B.Cu at (149.9, 78.7)
- moved C1 0.96 mm to (156.5, 86.5)
- moved C2 0.95 mm to (156.5, 83.8)
- moved U1 0.13 mm to (149.9, 72.4)
Connections:
- P1 pad 3: /BLE_TX -> /BLE_RESET
- P1 pad 4: /BLE_RX -> /BLE_RTS
- P1 pad 6: /BLE_RTS -> /BLE_RX
- P1 pad 7: /BLE_RESET -> /BLE_TX
Routing:
- net /BLE_RESET: track 0.00 -> 41.5 mm
- net /BLE_TX: track 0.00 -> 29.7 mm
- net /BLE_RX: track 0.00 -> 29.0 mm
- net +VDD: track 0.00 -> 28.4 mm
- net /BLE_CTS: track 0.00 -> 28.3 mm
- net /BLE_RTS: track 0.00 -> 27.7 mm
- net GND-ISO: track 0.00 -> 11.5 mm, vias 0 -> 4
- net +3.3V: track 0.00 -> 4.34 mm
- net GND: track 0.00 -> 3.81 mm
- added copper zone on F.Cu, net GND-ISO
Other:
- net class Default: via_dia 0.8 -> 0.6; via_drill 0.4 -> 0.3
- rule trace_min: 0.2 -> 0.25
- rule via_min_size: 0.4 -> 0.6
- board text added: "BGM111 Breakout"
- board text added: "CTS"
- board text added: "NOWAE026-0"
- board text added: "RESET"
- board text added: "RTS"
- board text added: "RX"
- board text added: "TX"
- board text added: "designed by"

Commit message: Ended PCB design (nowae026)
Parts:
- added G***: LOGO, EXTLOGO:LOGO_OSH_10MM_FSILK, B.Cu at (145.0, 87.7)
- added G***: LOGO, EXTLOGO:LOGO_CC-BY-SA_10MM_FSILK, B.Cu at (154.7, 86.1)
- moved G*** 1.87 mm to (149.9, 76.9)
Routing:
- net GND-ISO: vias 4 -> 44
Other:
- rule trace_min: 0.25 -> 0.2
- board text added: "www.nowae.it"
