File: 05-Layout/nowae027/nowae027-0/nowae027.kicad_pcb (KiCad board)
At the start: 2 copper layers, 17.8 x 30.5 mm, 11 parts, among them P1 CONN, P2 OLED

Commit message: Ended routing (nowae027)
Parts:
- added G***: LOGO, LOGO:LOGO_NOWAE_15MM_FSILK, B.Cu at (143.4, 99.7)
- added G***: LOGO, EXTLOGO:LOGO_OSH_5MM_FSILK, B.Cu at (143.6, 95.7)
- added G***: LOGO, LOGO:LOGO_NOWAE_5MM_FSILK, F.Cu at (143.4, 102.1)
- added VAL**: FIDUCIALMARK_1MM_2MM, MECHANICAL:FIDUCIALMARK_1MM_2MM, B.Cu at (135.9, 102.9)
- added VAL**: FIDUCIALMARK_1MM_2MM, MECHANICAL:FIDUCIALMARK_1MM_2MM, B.Cu at (151.1, 74.9)
- added VAL?: DISPLAY-RAYSTAR-REX004864A_ONLY3D, DISPLAY:DISPLAY-RAYSTAR-REX004864A_ONLY3D, F.Cu at (143.5, 90.1)
- moved C1 68.2 mm to (139.7, 81.9)
- moved C2 68.2 mm to (139.7, 79.4)
- moved P1 68.2 mm to (143.5, 76.2)
- moved R2 68.2 mm to (147.3, 79.4)
- moved R3 68.2 mm to (147.3, 81.9)
- moved C3 68.2 mm to (137.8, 85.7)
- moved C6 68.2 mm to (149.2, 85.7)
- moved C4 68.2 mm to (140.3, 85.7)
- moved C5 68.2 mm to (146.7, 85.7)
- moved P2 68.2 mm to (143.4, 91.4)
- moved R1 68.2 mm to (144.1, 85.7)
Routing:
- net +3.3V: track 0.00 -> 35.5 mm
- net /OLED_SDA: track 0.00 -> 23.7 mm, vias 0 -> 1
- net /OLED_SCL: track 0.00 -> 20.7 mm, vias 0 -> 1
- net GND: track 0.00 -> 19.1 mm
- net /OLED_RESET: track 0.00 -> 15.6 mm, vias 0 -> 1
- net Net-(C3-Pad2): track 0.00 -> 7.91 mm
- net Net-(C4-Pad2): track 0.00 -> 7.87 mm
- net Net-(P2-Pad12): track 0.00 -> 6.25 mm
- net Net-(C6-Pad2): track 0.00 -> 4.78 mm
- net Net-(C3-Pad1): track 0.00 -> 4.72 mm
- net Net-(C5-Pad2): track 0.00 -> 4.52 mm
- net Net-(C4-Pad1): track 0.00 -> 4.28 mm
Other:
- board text added: "NOWAE027-0"
- board text added: "www.nowae.it"
