File: 05-Layout/nowae012/nowae012-0/nowae012.kicad_pcb (KiCad board)
At the start: 2 copper layers, 38 x 11 mm, 32 parts, among them P1 USB3.1-C, P2 USB3.1-C, Q1 STL6P3LLH6, U1 STUSB4500QTR

Commit message: WiP: schematic and layout (nowae012-0)
Parts:
- removed TP3, TP4: TEST_POINT, MISC:TESTPOINT-0.5MM-SMD
- added P3: I2C, CONNECTOR:CONN-PAD-3x1-1.27, B.Cu at (11.6, 10.0)
- D1, D3: value ESDA25P35-1U1M -> ESDA25P35
- D2: footprint SOT:SOT23-3 -> SOT:SOT323-3
- U1: value STUSB4500QTR -> STUSB4500LQTR
- moved TP5 3.00 mm to (20.2, 11.3)
- moved G*** 0.70 mm to (14.8, 6.30)
- moved G*** 0.70 mm to (22.5, 6.30)
- moved R2 0.50 mm to (21.9, 8.30)
- moved R7 0.50 mm to (21.1, 2.20)
- moved C1 0.50 mm to (12.3, 3.40)
- moved C2 0.50 mm to (17.7, 4.50)
- moved C3 0.50 mm to (16.8, 4.50)
- moved C4 0.50 mm to (22.9, 9.70)
- moved C5 0.50 mm to (25.7, 3.40)
- moved D1 0.50 mm to (14.2, 3.90)
- moved D3 0.50 mm to (25.7, 8.00)
- moved DL1 0.50 mm to (23.5, 2.60)
- moved P1 0.50 mm to (4.90, 6.00)
- moved P2 0.50 mm to (33.1, 6.00)
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Connections:
- net Net-(C3-Pad1) renamed /+2V7
- Q1 pad 3: Net-(Q1-Pad3) -> Net-(C1-Pad2)
Routing:
- net Net-(P3-Pad2): track 4.05 -> 6.64 mm
- net GND: track 33.2 -> 30.9 mm
- net Net-(TP5-Pad1): track 5.56 -> 3.52 mm
- net Net-(P3-Pad1): track 4.43 -> 6.01 mm
- net Net-(C1-Pad2): track 18.6 -> 19.2 mm
Other:
- board size 38 x 11 mm -> 38 x 12 mm
